Commit message: Add matched collision hulls, Inspect Robots embodiment, and scene view/edit CLI
- Collision: CoACD convex decomposition per link (scripts/make_collision_meshes.py),
  one URDF collision per hull; scripts/check_collision.py measures the match by raycast
  (91-99.8% of surface within 2 mm).
- yam_sim embodiment for inspect-robots: top_cam plus left/right wrist cameras,
  14-D joint state/action matching the real yam_arms contract; -E scene= loads a saved scene.
- yam-sim CLI: `view` runs a scene with the arms held in the ready pose; `edit` opens it in
  Isaac Sim with Play/Pause/Stop/Save in a panel and saves only the environment.
- Wrist cameras follow the grippers; gravity compensation holds the arms.

Co-Authored-By: Claude Opus 5.5 <noreply@anthropic.com>

File: assets/yam/yam_sim.urdf (robot description, URDF)
Before this commit: robot yam, 9 links, 8 joints
Links:
- link base: geometry collision mesh filename=collision/base/base_000.stl scale=1 1 1; collision mesh filename=collision/base/base_001.stl scale=1 1 1
- link gripper: geometry collision mesh filename=collision/gripper/gripper_000.stl scale=1 1 1; collision mesh filename=collision/gripper/gripper_001.stl scale=1 1 1
- link link1: geometry collision mesh filename=collision/link1/link1_000.stl scale=1 1 1; collision mesh filename=collision/link1/link1_001.stl scale=1 1 1
- link link2: geometry collision mesh filename=collision/link2/link2_000.stl scale=1 1 1; collision mesh filename=collision/link2/link2_001.stl scale=1 1 1
- link link3: geometry collision mesh filename=collision/link3/link3_000.stl scale=1 1 1; collision mesh filename=collision/link3/link3_001.stl scale=1 1 1
- link link4: geometry collision mesh filename=collision/link4/link4_000.stl scale=1 1 1; collision mesh filename=collision/link4/link4_001.stl scale=1 1 1
- link link5: geometry collision mesh filename=collision/link5/link5_000.stl scale=1 1 1; collision mesh filename=collision/link5/link5_001.stl scale=1 1 1
- link tip_left: geometry collision mesh filename=collision/tip_left/tip_left_000.stl scale=1 1 1; collision mesh filename=collision/tip_left/tip_left_001.stl scale=1 1 1
- link tip_right: geometry collision mesh filename=collision/tip_right/tip_right_000.stl scale=1 1 1; collision mesh filename=collision/tip_right/tip_right_001.stl scale=1 1 1
